Commit message: Fix Kuavo S54 head joints for visualization

File: src/holosoma_retargeting/holosoma_retargeting/models/kuavo_s54/kuavo_s54_29dof.urdf (robot description, URDF)
Before this commit: robot biped_s54, 35 links, 34 joints
Joints:
- joint zhead_1_joint: type fixed -> revolute
- joint zhead_2_joint: type fixed -> revolute
